Commit message: chore: refine constants and xacro parameterization from review feedback
Agent-Logs-Url: https://github.com/Rajasbhatnagar/warehouse_amr_ros2/sessions/6b2ca223-9ea6-4890-8749-06078801fd9c

Co-authored-by: Rajasbhatnagar <151607014+Rajasbhatnagar@users.noreply.github.com>

File: ros2_ws/src/amr_description/urdf/base.xacro (robot description, xacro)
@@ -1,5 +1,5 @@
 <?xml version="1.0"?>
 <robot xmlns:xacro="http://www.ros.org/wiki/xacro">
-  <xacro:macro name="amr_base" params="base_length base_width base_height wheel_radius wheel_width wheel_separation">
+  <xacro:macro name="amr_base" params="base_length base_width base_height wheel_radius wheel_width wheel_separation caster_offset_ratio">
     <link name="base_link">
       <visual>
@@ -76,5 +76,5 @@
       <parent link="base_link"/>
       <child link="caster_link"/>
-      <origin xyz="-${base_length/2.5} 0 0.04"/>
+      <origin xyz="-${base_length/caster_offset_ratio} 0 0.04"/>
     </joint>
   </xacro:macro>

File: ros2_ws/src/amr_description/urdf/robot.urdf.xacro (robot description, xacro)
@@ -8,4 +8,5 @@
   <xacro:property name="wheel_width" value="0.04"/>
   <xacro:property name="wheel_separation" value="0.34"/>
+  <xacro:property name="caster_offset_ratio" value="2.5"/>
   <xacro:include filename="$(find amr_description)/urdf/materials.xacro"/>
   <xacro:include filename="$(find amr_description)/urdf/base.xacro"/>
@@ -18,5 +19,6 @@
     wheel_radius="${wheel_radius}"
     wheel_width="${wheel_width}"
-    wheel_separation="${wheel_separation}"/>
+    wheel_separation="${wheel_separation}"
+    caster_offset_ratio="${caster_offset_ratio}"/>
   <xacro:amr_sensors base_length="${base_length}" base_height="${base_height}"/>
   <xacro:if value="$(arg use_ros2_control)">

Commit message: fix: harden perception rate handling and PID anti-windup
Agent-Logs-Url: https://github.com/Rajasbhatnagar/warehouse_amr_ros2/sessions/6b2ca223-9ea6-4890-8749-06078801fd9c

Co-authored-by: Rajasbhatnagar <151607014+Rajasbhatnagar@users.noreply.github.com>

File: ros2_ws/src/amr_description/urdf/base.xacro (robot description, xacro)
@@ -1,5 +1,5 @@
 <?xml version="1.0"?>
 <robot xmlns:xacro="http://www.ros.org/wiki/xacro">
-  <xacro:macro name="amr_base" params="base_length base_width base_height wheel_radius wheel_width wheel_separation caster_offset_ratio">
+  <xacro:macro name="amr_base" params="base_length base_width base_height wheel_radius wheel_width wheel_separation caster_offset_ratio caster_radius">
     <link name="base_link">
       <visual>
@@ -62,9 +62,9 @@
     <link name="caster_link">
       <visual>
-        <geometry><sphere radius="0.04"/></geometry>
+        <geometry><sphere radius="${caster_radius}"/></geometry>
         <material name="light_gray"/>
       </visual>
       <collision>
-        <geometry><sphere radius="0.04"/></geometry>
+        <geometry><sphere radius="${caster_radius}"/></geometry>
       </collision>
       <inertial>
@@ -76,5 +76,5 @@
       <parent link="base_link"/>
       <child link="caster_link"/>
-      <origin xyz="-${base_length/caster_offset_ratio} 0 0.04"/>
+      <origin xyz="-${base_length/caster_offset_ratio} 0 ${caster_radius}"/>
     </joint>
   </xacro:macro>

File: ros2_ws/src/amr_description/urdf/robot.urdf.xacro (robot description, xacro)
@@ -9,4 +9,6 @@
   <xacro:property name="wheel_separation" value="0.34"/>
   <xacro:property name="caster_offset_ratio" value="2.5"/>
+  <xacro:property name="caster_radius" value="0.04"/>
+  <xacro:property name="camera_front_offset" value="0.05"/>
   <xacro:include filename="$(find amr_description)/urdf/materials.xacro"/>
   <xacro:include filename="$(find amr_description)/urdf/base.xacro"/>
@@ -20,6 +22,10 @@
     wheel_width="${wheel_width}"
     wheel_separation="${wheel_separation}"
-    caster_offset_ratio="${caster_offset_ratio}"/>
-  <xacro:amr_sensors base_length="${base_length}" base_height="${base_height}"/>
+    caster_offset_ratio="${caster_offset_ratio}"
+    caster_radius="${caster_radius}"/>
+  <xacro:amr_sensors
+    base_length="${base_length}"
+    base_height="${base_height}"
+    camera_front_offset="${camera_front_offset}"/>
   <xacro:if value="$(arg use_ros2_control)">
     <xacro:amr_ros2_control

File: ros2_ws/src/amr_description/urdf/sensors.xacro (robot description, xacro)
@@ -1,5 +1,5 @@
 <?xml version="1.0"?>
 <robot xmlns:xacro="http://www.ros.org/wiki/xacro">
-  <xacro:macro name="amr_sensors" params="base_length base_height">
+  <xacro:macro name="amr_sensors" params="base_length base_height camera_front_offset">
     <link name="lidar_link">
       <visual>
@@ -36,5 +36,5 @@
       <parent link="base_link"/>
       <child link="camera_link"/>
-      <origin xyz="${base_length/2.0 - 0.05} 0 ${base_height + 0.08}"/>
+      <origin xyz="${base_length/2.0 - camera_front_offset} 0 ${base_height + 0.08}"/>
     </joint>
   </xacro:macro>
